Commit message: renamed hector_quadrotor_urdf package to hector_quadrotor_description to follow ROS standards and moved plugin configuration files to hector_quadrotor_gazebo/urdf

File: hector_quadrotor_description/urdf/quadrotor_downward_cam.urdf.xacro (robot description, xacro)
@@ -6,5 +6,5 @@
     <xacro:property name="M_PI" value="3.1415926535897931" />
     <!-- Included URDF Files -->
-    <xacro:include filename="$(find hector_quadrotor_urdf)/urdf/quadrotor_base.urdf.xacro" />
+    <xacro:include filename="$(find hector_quadrotor_description)/urdf/quadrotor_base.urdf.xacro" />
     <!-- Instantiate quadrotor_base_macro once (has no parameters atm) -->
     <xacro:quadrotor_base_macro />

File: hector_quadrotor_description/urdf/quadrotor_hokuyo_utm30lx.urdf.xacro (robot description, xacro)
@@ -6,12 +6,12 @@
     <xacro:property name="M_PI" value="3.1415926535897931" />
     <!-- Included URDF Files -->
-    <xacro:include filename="$(find hector_quadrotor_urdf)/urdf/quadrotor_base.urdf.xacro" />
+    <xacro:include filename="$(find hector_quadrotor_description)/urdf/quadrotor_base.urdf.xacro" />
     <!-- Instantiate quadrotor_base_macro once (has no parameters atm) -->
     <xacro:quadrotor_base_macro />
     <!-- Hokuyo UTM-30LX mounted upside down below the quadrotor body -->
-    <!-- xacro:include filename="$(find hector_sensors_description)/urdf/hokuyo_utm30lx.urdf.xacro" />
+    <xacro:include filename="$(find hector_sensors_description)/urdf/hokuyo_utm30lx.urdf.xacro" />
     <xacro:hokuyo_utm30lx name="laser0" parent="base_link" ros_topic="scan" update_rate="40" ray_count="1081" min_angle="135" max_angle="-135">
       <origin xyz="0.0 0.0 -0.097" rpy="${M_PI} 0 0"/>
-    </xacro:hokuyo_utm30lx -->
+    </xacro:hokuyo_utm30lx>
     <!-- Forward facing camera -->
     <xacro:include filename="$(find hector_sensors_description)/urdf/generic_camera.urdf.xacro" />

File: hector_quadrotor_description/urdf/quadrotor_with_asus.urdf.xacro (robot description, xacro)
@@ -6,5 +6,5 @@
     <xacro:property name="M_PI" value="3.1415926535897931" />
     <!-- Included URDF Files -->
-    <xacro:include filename="$(find hector_quadrotor_urdf)/urdf/quadrotor_base.urdf.xacro" />
+    <xacro:include filename="$(find hector_quadrotor_description)/urdf/quadrotor_base.urdf.xacro" />
     <!-- Instantiate quadrotor_base_macro once (has no parameters atm) -->
     <xacro:quadrotor_base_macro />

File: hector_quadrotor_description/urdf/quadrotor_with_asus_with_hokuyo_utm30lx.urdf.xacro (robot description, xacro)
@@ -6,5 +6,5 @@
     <xacro:property name="M_PI" value="3.1415926535897931" />
     <!-- Included URDF Files -->
-    <xacro:include filename="$(find hector_quadrotor_urdf)/urdf/quadrotor_base.urdf.xacro" />
+    <xacro:include filename="$(find hector_quadrotor_description)/urdf/quadrotor_base.urdf.xacro" />
     <!-- Instantiate quadrotor_base_macro once (has no parameters atm) -->
     <xacro:quadrotor_base_macro />
@@ -14,8 +14,8 @@
       <origin xyz="0.0 0.0 -0.097" rpy="${M_PI} 0 0"/>
     </xacro:hokuyo_utm30lx>
-    <!-- Forward facing camera -->
-    <xacro:include filename="$(find hector_sensors_description)/urdf/generic_camera.urdf.xacro" />
-    <xacro:generic_camera name="front_cam" parent="base_link" ros_topic="camera/image" cam_info_topic="camera/camera_info" update_rate="10" res_x="320" res_y="240" image_format="R8G8B8" hfov="90">
-      <origin xyz="0.05 0.0 -0.06" rpy="0 0 0"/>
-    </xacro:generic_camera>
+    <!-- Asus Xiton Live Pro -->
+    <xacro:include filename="$(find hector_sensors_description)/urdf/asus_camera.urdf.xacro" />
+    <xacro:asus_camera name="camera" parent="base_link">
+      <origin xyz="0.1 0.0 -0.03" rpy="0 ${M_PI/9} 0"/>
+    </xacro:asus_camera>
 </robot>
