Commit message: Modified location of camera

File: hector_quadrotor_description/urdf/quadrotor_base.urdf.xacro (robot description, xacro)
@@ -24,4 +24,18 @@
       </collision>
     </link>
+    <!-- additional link for attaching camera -->
+    <link name="add_link">
+      <visual>
+        <geometry>
+          <cylinder length="0.6" radius="0.004"/>
+        </geometry>
+        <origin rpy="0 1.57075 0.785375" xyz="0 0 0"/>
+      </visual>
+    </link>
+    <joint name="base_to_add_link" type="fixed">
+      <parent link="base_link"/>
+      <child link="add_link"/>
+      <origin xyz="0 0 0"/>
+    </joint>
     <!-- Sonar height sensor -->
     <xacro:sonar_sensor name="sonar" parent="base_link" ros_topic="sonar_height" update_rate="10" min_range="0.03" max_range="3.0" field_of_view="${40*pi/180}" ray_count="3">

File: hector_quadrotor_description/urdf/quadrotor_hokuyo_utm30lx.urdf.xacro (robot description, xacro)
@@ -9,10 +9,10 @@
     <xacro:include filename="$(find hector_sensors_description)/urdf/hokuyo_utm30lx.urdf.xacro" />
     <xacro:hokuyo_utm30lx name="laser0" parent="base_link" ros_topic="scan" update_rate="40" ray_count="1081" min_angle="-135" max_angle="135">
-      <origin xyz="0.0 0.0 -0.097" rpy="${M_PI} 0 0"/>
+      <origin xyz="0.0 0.0 -0.087" rpy="${M_PI} 0 0"/>
     </xacro:hokuyo_utm30lx>
     <!-- Forward facing camera -->
     <xacro:include filename="$(find hector_sensors_description)/urdf/generic_camera.urdf.xacro" />
-    <xacro:generic_camera name="front_cam" parent="base_link" ros_topic="camera/image" cam_info_topic="camera/camera_info" update_rate="10" res_x="320" res_y="240" image_format="R8G8B8" hfov="90">
-      <origin xyz="0.05 0.0 -0.06" rpy="0 0 0"/>
+    <xacro:generic_camera name="front_cam" parent="add_link" ros_topic="camera/image" cam_info_topic="camera/camera_info" update_rate="10" res_x="320" res_y="240" image_format="R8G8B8" hfov="90">
+      <origin xyz="0.21142 0.21142 0" rpy="0 0 0.785375"/>
     </xacro:generic_camera>
 </robot>

File: hector_quadrotor_description/urdf/quadrotor_with_cam.urdf.xacro (robot description, xacro)
@@ -8,6 +8,6 @@
     <!-- Forward facing camera -->
     <xacro:include filename="$(find hector_sensors_description)/urdf/generic_camera.urdf.xacro" />
-    <xacro:generic_camera name="front_cam" parent="base_link" ros_topic="camera/image" cam_info_topic="camera/camera_info" update_rate="10" res_x="320" res_y="240" image_format="R8G8B8" hfov="90">
-      <origin xyz="0.05 0.0 -0.06" rpy="0 0 0"/>
+    <xacro:generic_camera name="front_cam" parent="add_link" ros_topic="camera/image" cam_info_topic="camera/camera_info" update_rate="10" res_x="320" res_y="240" image_format="R8G8B8" hfov="90">
+      <origin xyz="0.21142 0.21142 0" rpy="0 0 0.785375"/>
     </xacro:generic_camera>
 </robot>
