Commit message: hector_quadrotor_controller/hector_quadrotor_controller_gazebo:
 * using ROS parameters to configure state topics
 * use controller_manager in gazebo_ros_control instead of running standalone pose_controller
 * keep track of which controller is enabled() in QuadrotorInterface class
 * ...

File: hector_quadrotor_gazebo/urdf/quadrotor_controller.gazebo.xacro (robot description, xacro)
@@ -1,38 +1,9 @@
 <?xml version="1.0"?>
 <robot xmlns:xacro="http://ros.org/wiki/xacro">
-  <!-- Quadrotor Controller Plugin -->
-  <xacro:macro name="quadrotor_controller" params="state_topic imu_topic">
+  <xacro:macro name="quadrotor_controller">
     <gazebo>
-      <plugin name="quadrotor_controller" filename="libgazebo_rtt_plugin.so">
-        <updateRate>100.0</updateRate>
-        <import>quadro</import>
-        <component>Controller</component>
-        <configuration>$(find quadro)/conf/controller.cpf</configuration>
-        <port><name>sonar_height</name></port>
-        <port><name>command_velocity</name><topic>cmd_vel</topic></port>
-        <port><name>rc</name><topic>rc</topic></port>
-        <port><name>state</name><topic>${state_topic}</topic><queue_size>10</queue_size></port>
-        <port><name>imu</name><topic>${imu_topic}</topic><queue_size>10</queue_size></port>
-        <port><name>motor_status</name></port>
-        <port><name>height</name><queue_size>10</queue_size></port>
-        <port><name>motor_input</name><topic>input/motor</topic><queue_size>10</queue_size></port>
-        <port><name>motor_output</name><topic>motor_pwm</topic><queue_size>10</queue_size></port>
-        <port><name>attitude_command</name><topic>command/attitude</topic><queue_size>1</queue_size></port>
-        <port><name>attitude_input</name><topic>input/attitude</topic><queue_size>10</queue_size></port>
-        <port><name>attitude_rate_input</name><topic>input/rate</topic><queue_size>10</queue_size></port>
-        <port><name>velocity_command</name><topic>command/velocity</topic><queue_size>1</queue_size></port>
-        <port><name>velocity_input</name><topic>input/velocity</topic><queue_size>10</queue_size></port>
-        <port><name>position_command</name><topic>command/position</topic><queue_size>1</queue_size></port>
-        <port><name>position_input</name><topic>input/position</topic><queue_size>10</queue_size></port>
-        <port><name>heading_command</name><topic>command/heading</topic><queue_size>1</queue_size></port>
-        <port><name>heading_input</name><topic>input/heading</topic><queue_size>10</queue_size></port>
-        <port><name>heading_rate_command</name><topic>command/turnrate</topic><queue_size>1</queue_size></port>
-        <port><name>heading_rate_input</name><topic>input/turnrate</topic><queue_size>10</queue_size></port>
-        <port><name>height_command</name><topic>command/height</topic><queue_size>1</queue_size></port>
-        <port><name>height_input</name><topic>input/height</topic><queue_size>10</queue_size></port>
-        <port><name>height_rate_command</name><topic>command/climbrate</topic><queue_size>1</queue_size></port>
-        <port><name>height_rate_input</name><topic>input/climbrate</topic><queue_size>10</queue_size></port>
-        <port><name>height_rate_output</name><topic>output/climbrate</topic><queue_size>10</queue_size></port>
-        <port><name>command_velocity_input</name><topic>input/cmd_vel</topic><queue_size>10</queue_size></port>
+      <plugin name="quadrotor_controller" filename="libgazebo_ros_control.so">
+        <!-- <controlPeriod>0.01</controlPeriod> -->
+        <robotSimType>hector_quadrotor_controller_gazebo/QuadrotorHardwareSim</robotSimType>
       </plugin>
     </gazebo>
