Commit message: hector_quadrotor_gazebo: a few fixes for RTT integration in hector_quadrotor. Added urdf macro for rtt_gazebo_plugin macro.

File: hector_quadrotor_gazebo/urdf/quadrotor_rtt_controller.gazebo.xacro (robot description, xacro)
@@ -2,5 +2,5 @@
 <robot xmlns:xacro="http://ros.org/wiki/xacro">
   <!-- Quadrotor Controller Plugin -->
-  <xacro:macro name="quadrotor_controller" params="state_topic imu_topic">
+  <xacro:macro name="quadrotor_rtt_controller" params="state_topic imu_topic">
     <gazebo>
       <plugin name="quadrotor_controller" filename="libgazebo_rtt_plugin.so">
